Commit message: Modified package name in each file.

File: urdf/rohand_left.urdf (robot description, URDF)
Before this commit: robot rohand_left, 26 links, 25 joints
Links:
- link base_link: geometry collision mesh filename=package://rohand_urdf_ros2/meshes_l/base_link.STL; visual mesh filename=package://rohand_urdf_ros2/meshes_l/base_link.STL
- link if_connecting_link: geometry collision mesh filename=package://rohand_urdf_ros2/meshes_l/if_connecting_link.STL; visual mesh filename=package://rohand_urdf_ros2/meshes_l/if_connecting_link.STL
- link if_distal_link: geometry collision mesh filename=package://rohand_urdf_ros2/meshes_l/if_distal_link.STL; visual mesh filename=package://rohand_urdf_ros2/meshes_l/if_distal_link.STL
- link if_proximal_link: geometry collision mesh filename=package://rohand_urdf_ros2/meshes_l/if_proximal_link.STL; visual mesh filename=package://rohand_urdf_ros2/meshes_l/if_proximal_link.STL
- link if_slider_abpart_link: geometry collision mesh filename=package://rohand_urdf_ros2/meshes_l/if_slider_abpart_link.S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; visual mesh filename=package://rohand_urdf_ros2/meshes_l/if_slider_abpart_link.S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
- link if_slider_link: geometry collision mesh filename=package://rohand_urdf_ros2/meshes_l/if_slider_link.STL; visual mesh filename=package://rohand_urdf_ros2/meshes_l/if_slider_link.STL
- link lf_connecting_link: geometry collision mesh filename=package://rohand_urdf_ros2/meshes_l/lf_connecting_link.STL; visual mesh filename=package://rohand_urdf_ros2/meshes_l/lf_connecting_link.STL
- link lf_distal_link: geometry collision mesh filename=package://rohand_urdf_ros2/meshes_l/lf_distal_link.STL; visual mesh filename=package://rohand_urdf_ros2/meshes_l/lf_distal_link.STL
- link lf_proximal_link: geometry collision mesh filename=package://rohand_urdf_ros2/meshes_l/lf_proximal_link.STL; visual mesh filename=package://rohand_urdf_ros2/meshes_l/lf_proximal_link.STL
- link lf_slider_abpart_link: geometry collision mesh filename=package://rohand_urdf_ros2/meshes_l/lf_slider_abpart_link.S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; visual mesh filename=package://rohand_urdf_ros2/meshes_l/lf_slider_abpart_link.S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
- link lf_slider_link: geometry collision mesh filename=package://rohand_urdf_ros2/meshes_l/lf_slider_link.STL; visual mesh filename=package://rohand_urdf_ros2/meshes_l/lf_slider_link.STL
- link mf_connecting_link: geometry collision mesh filename=package://rohand_urdf_ros2/meshes_l/mf_connecting_link.STL; visual mesh filename=package://rohand_urdf_ros2/meshes_l/mf_connecting_link.STL
- link mf_distal_link: geometry collision mesh filename=package://rohand_urdf_ros2/meshes_l/mf_distal_link.STL; visual mesh filename=package://rohand_urdf_ros2/meshes_l/mf_distal_link.STL
- link mf_proximal_link: geometry collision mesh filename=package://rohand_urdf_ros2/meshes_l/mf_proximal_link.STL; visual mesh filename=package://rohand_urdf_ros2/meshes_l/mf_proximal_link.STL
- link mf_slider_abpart_link: geometry collision mesh filename=package://rohand_urdf_ros2/meshes_l/mf_slider_abpart_link.S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; visual mesh filename=package://rohand_urdf_ros2/meshes_l/mf_slider_abpart_link.S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
- link mf_slider_link: geometry collision mesh filename=package://rohand_urdf_ros2/meshes_l/mf_slider_link.STL; visual mesh filename=package://rohand_urdf_ros2/meshes_l/mf_slider_link.STL
- link rf_connecting_link: geometry collision mesh filename=package://rohand_urdf_ros2/meshes_l/rf_connecting_link.STL; visual mesh filename=package://rohand_urdf_ros2/meshes_l/rf_connecting_link.STL
- link rf_distal_link: geometry collision mesh filename=package://rohand_urdf_ros2/meshes_l/rf_distal_link.STL; visual mesh filename=package://rohand_urdf_ros2/meshes_l/rf_distal_link.STL
- link rf_proximal_link: geometry collision mesh filename=package://rohand_urdf_ros2/meshes_l/rf_proximal_link.STL; visual mesh filename=package://rohand_urdf_ros2/meshes_l/rf_proximal_link.STL
- link rf_slider_abpart_link: geometry collision mesh filename=package://rohand_urdf_ros2/meshes_l/rf_slider_abpart_link.S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; visual mesh filename=package://rohand_urdf_ros2/meshes_l/rf_slider_abpart_link.S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
- link rf_slider_link: geometry collision mesh filename=package://rohand_urdf_ros2/meshes_l/rf_slider_link.STL; visual mesh filename=package://rohand_urdf_ros2/meshes_l/rf_slider_link.STL
- link th_connecting_link: geometry collision mesh filename=package://rohand_urdf_ros2/meshes_l/th_connecting_link.STL; visual mesh filename=package://rohand_urdf_ros2/meshes_l/th_connecting_link.STL
- link th_distal_link: geometry collision mesh filename=package://rohand_urdf_ros2/meshes_l/th_distal_link.STL; visual mesh filename=package://rohand_urdf_ros2/meshes_l/th_distal_link.STL
- link th_proximal_link: geometry collision mesh filename=package://rohand_urdf_ros2/meshes_l/th_proximal_link.STL; visual mesh filename=package://rohand_urdf_ros2/meshes_l/th_proximal_link.STL
- link th_root_link: geometry collision mesh filename=package://rohand_urdf_ros2/meshes_l/th_root_link.STL; visual mesh filename=package://rohand_urdf_ros2/meshes_l/th_root_link.STL
- link th_slider_link: geometry collision mesh filename=package://rohand_urdf_ros2/meshes_l/th_slider_link.STL; visual mesh filename=package://rohand_urdf_ros2/meshes_l/th_slider_link.STL

File: urdf/rohand_right.urdf (robot description, URDF)
Before this commit: robot rohand_right, 26 links, 25 joints
Links:
- link base_link: geometry collision mesh filename=package://rohand_urdf_ros2/meshes_r/base_link.STL; visual mesh filename=package://rohand_urdf_ros2/meshes_r/base_link.STL
- link if_connecting_link: geometry collision mesh filename=package://rohand_urdf_ros2/meshes_r/if_connecting_link.STL; visual mesh filename=package://rohand_urdf_ros2/meshes_r/if_connecting_link.STL
- link if_distal_link: geometry collision mesh filename=package://rohand_urdf_ros2/meshes_r/if_distal_link.STL; visual mesh filename=package://rohand_urdf_ros2/meshes_r/if_distal_link.STL
- link if_proximal_link: geometry collision mesh filename=package://rohand_urdf_ros2/meshes_r/if_proximal_link.STL; visual mesh filename=package://rohand_urdf_ros2/meshes_r/if_proximal_link.STL
- link if_slider_abpart_link: geometry collision mesh filename=package://rohand_urdf_ros2/meshes_r/if_slider_abpart_link.S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; visual mesh filename=package://rohand_urdf_ros2/meshes_r/if_slider_abpart_link.S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
- link if_slider_link: geometry collision mesh filename=package://rohand_urdf_ros2/meshes_r/if_slider_link.STL; visual mesh filename=package://rohand_urdf_ros2/meshes_r/if_slider_link.STL
- link lf_connecting_link: geometry collision mesh filename=package://rohand_urdf_ros2/meshes_r/lf_connecting_link.STL; visual mesh filename=package://rohand_urdf_ros2/meshes_r/lf_connecting_link.STL
- link lf_distal_link: geometry collision mesh filename=package://rohand_urdf_ros2/meshes_r/lf_distal_link.STL; visual mesh filename=package://rohand_urdf_ros2/meshes_r/lf_distal_link.STL
- link lf_proximal_link: geometry collision mesh filename=package://rohand_urdf_ros2/meshes_r/lf_proximal_link.STL; visual mesh filename=package://rohand_urdf_ros2/meshes_r/lf_proximal_link.STL
- link lf_slider_abpart_link: geometry collision mesh filename=package://rohand_urdf_ros2/meshes_r/lf_slider_abpart_link.S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; visual mesh filename=package://rohand_urdf_ros2/meshes_r/lf_slider_abpart_link.S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
- link lf_slider_link: geometry collision mesh filename=package://rohand_urdf_ros2/meshes_r/lf_slider_link.STL; visual mesh filename=package://rohand_urdf_ros2/meshes_r/lf_slider_link.STL
- link mf_connecting_link: geometry collision mesh filename=package://rohand_urdf_ros2/meshes_r/mf_connecting_link.STL; visual mesh filename=package://rohand_urdf_ros2/meshes_r/mf_connecting_link.STL
- link mf_distal_link: geometry collision mesh filename=package://rohand_urdf_ros2/meshes_r/mf_distal_link.STL; visual mesh filename=package://rohand_urdf_ros2/meshes_r/mf_distal_link.STL
- link mf_proximal_link: geometry collision mesh filename=package://rohand_urdf_ros2/meshes_r/mf_proximal_link.STL; visual mesh filename=package://rohand_urdf_ros2/meshes_r/mf_proximal_link.STL
- link mf_slider_abpart_link: geometry collision mesh filename=package://rohand_urdf_ros2/meshes_r/mf_slider_abpart_link.S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; visual mesh filename=package://rohand_urdf_ros2/meshes_r/mf_slider_abpart_link.S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
- link mf_slider_link: geometry collision mesh filename=package://rohand_urdf_ros2/meshes_r/mf_slider_link.STL; visual mesh filename=package://rohand_urdf_ros2/meshes_r/mf_slider_link.STL
- link rf_connecting_link: geometry collision mesh filename=package://rohand_urdf_ros2/meshes_r/rf_connecting_link.STL; visual mesh filename=package://rohand_urdf_ros2/meshes_r/rf_connecting_link.STL
- link rf_distal_link: geometry collision mesh filename=package://rohand_urdf_ros2/meshes_r/rf_distal_link.STL; visual mesh filename=package://rohand_urdf_ros2/meshes_r/rf_distal_link.STL
- link rf_proximal_link: geometry collision mesh filename=package://rohand_urdf_ros2/meshes_r/rf_proximal_link.STL; visual mesh filename=package://rohand_urdf_ros2/meshes_r/rf_proximal_link.STL
- link rf_slider_abpart_link: geometry collision mesh filename=package://rohand_urdf_ros2/meshes_r/rf_slider_abpart_link.S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; visual mesh filename=package://rohand_urdf_ros2/meshes_r/rf_slider_abpart_link.S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
- link rf_slider_link: geometry collision mesh filename=package://rohand_urdf_ros2/meshes_r/rf_slider_link.STL; visual mesh filename=package://rohand_urdf_ros2/meshes_r/rf_slider_link.STL
- link th_connecting_link: geometry collision mesh filename=package://rohand_urdf_ros2/meshes_r/th_connecting_link.STL; visual mesh filename=package://rohand_urdf_ros2/meshes_r/th_connecting_link.STL
- link th_distal_link: geometry collision mesh filename=package://rohand_urdf_ros2/meshes_r/th_distal_link.STL; visual mesh filename=package://rohand_urdf_ros2/meshes_r/th_distal_link.STL
- link th_proximal_link: geometry collision mesh filename=package://rohand_urdf_ros2/meshes_r/th_proximal_link.STL; visual mesh filename=package://rohand_urdf_ros2/meshes_r/th_proximal_link.STL
- link th_root_link: geometry collision mesh filename=package://rohand_urdf_ros2/meshes_r/th_root_link.STL; visual mesh filename=package://rohand_urdf_ros2/meshes_r/th_root_link.STL
- link th_slider_link: geometry collision mesh filename=package://rohand_urdf_ros2/meshes_r/th_slider_link.STL; visual mesh filename=package://rohand_urdf_ros2/meshes_r/th_slider_link.STL

Commit message: Modified position of base_link axis

File: urdf/rohand_left.urdf (robot description, URDF)
Before this commit: robot rohand_left, 26 links, 25 joints
Links:
- link base_link: mass 0.0559618850522869 -> 0.0559618850523164
- link th_slider_link: mass 0.000966918573679237 -> 0.000966918573679238
Joints:
- joint if_connecting_link: origin xyz=-0.11976 0.03521 0.0028896 rpy=0 0 0 -> xyz=-0.11976 0.03521 0.0067299 rpy=0 0 0
- joint if_proximal_link: origin xyz=-0.11211 0.037738 -0.0018032 rpy=0 0 0 -> xyz=-0.11211 0.037738 0.0020371 rpy=0 0 0
- joint if_slider_link: origin xyz=-0.074396 0.026655 -0.0097434 rpy=0 0 0 -> xyz=-0.074396 0.026655 -0.0059032 rpy=0 0 0
- joint lf_connecting_link: origin xyz=-0.11723 -0.027174 0.0045247 rpy=0 0 0 -> xyz=-0.11723 -0.027174 0.008365 rpy=0 0 0
- joint lf_proximal_link: origin xyz=-0.11032 -0.022406 0.00045133 rpy=0 0 0 -> xyz=-0.11032 -0.022406 0.0042916 rpy=0 0 0
- joint lf_slider_link: origin xyz=-0.070847 -0.024182 -0.0087399 rpy=0 0 0 -> xyz=-0.070847 -0.024182 -0.0048997 rpy=0 0 0
- joint mf_connecting_link: origin xyz=-0.12334 0.014341 0.0075259 rpy=0 0 0 -> xyz=-0.12334 0.014341 0.011366 rpy=0 0 0
- joint mf_proximal_link: origin xyz=-0.11587 0.017792 0.0031262 rpy=0 0 0 -> xyz=-0.11587 0.017792 0.0069665 rpy=0 0 0
- joint mf_slider_link: origin xyz=-0.076974 0.010077 -0.0054756 rpy=0 0 0 -> xyz=-0.076974 0.010077 -0.0016353 rpy=0 0 0
- joint rf_connecting_link: origin xyz=-0.11723 -0.027174 0.0045247 rpy=0 0 0 -> xyz=-0.11723 -0.027174 0.008365 rpy=0 0 0
- joint rf_proximal_link: origin xyz=-0.11364 -0.0022565 0.0023761 rpy=0 0 0 -> xyz=-0.11364 -0.0022565 0.0062163 rpy=0 0 0
- joint rf_slider_link: origin xyz=-0.074498 -0.0072492 -0.0062204 rpy=0 0 0 -> xyz=-0.074498 -0.0072492 -0.0023801 rpy=0 0 0
- joint th_root_link: origin xyz=-0.024656 0.019554 -0.022107 rpy=0 0 0 -> xyz=-0.024656 0.019554 -0.018266 rpy=0 0 0
- joint th_slider_link: axis -0.761977793105663 0.630282689066857 -0.148773568473957 -> -0.76198 0.63028 -0.14877; origin xyz=-0.0076999999999972 0.00276927591433551 -0.000236666241639902 rpy=0 -1.3519569747769 -0.0320343601595158 -> xyz=-0.0077 0.0027693 -0.00023667 rpy=0 -1.352 -0.032034
