Commit message: joints distinguish between left and right hands

File: urdf/rohand_left.urdf (robot description, URDF)
Before this commit: robot rohand_left, 26 links, 25 joints
Links:
- removed link base_link
- removed link if_connecting_link
- removed link if_distal_link
- removed link if_proximal_link
- removed link if_slider_abpart_link
- removed link if_slider_link
- removed link lf_connecting_link
- removed link lf_distal_link
- removed link lf_proximal_link
- removed link lf_slider_abpart_link
- removed link lf_slider_link
- removed link mf_connecting_link
- removed link mf_distal_link
- removed link mf_proximal_link
- removed link mf_slider_abpart_link
- removed link mf_slider_link
- removed link rf_connecting_link
- removed link rf_distal_link
- removed link rf_proximal_link
- removed link rf_slider_abpart_link
- removed link rf_slider_link
- removed link th_connecting_link
- removed link th_distal_link
- removed link th_proximal_link
- removed link th_root_link
- removed link th_slider_link
- added link l_base_link, mass 0.0559618850523164; collision mesh filename=package://rohand_urdf_ros2/meshes_l/base_link.STL; visual mesh filename=package://rohand_urdf_ros2/meshes_l/base_link.STL
- added link l_if_connecting_link, mass 0.000197692348310411; collision mesh filename=package://rohand_urdf_ros2/meshes_l/if_connecting_link.STL; visual mesh filename=package://rohand_urdf_ros2/meshes_l/if_connecting_link.STL
- added link l_if_distal_link, mass 0.0042269383122795; collision mesh filename=package://rohand_urdf_ros2/meshes_l/if_distal_link.STL; visual mesh filename=package://rohand_urdf_ros2/meshes_l/if_distal_link.STL
- added link l_if_proximal_link, mass 0.00154987032874225; collision mesh filename=package://rohand_urdf_ros2/meshes_l/if_proximal_link.STL; visual mesh filename=package://rohand_urdf_ros2/meshes_l/if_proximal_link.STL
- added link l_if_slider_abpart_link, mass 0.000419595822746572; collision mesh filename=package://rohand_urdf_ros2/meshes_l/if_slider_abpart_link.S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; visual mesh filename=package://rohand_urdf_ros2/meshes_l/if_slider_abpart_link.S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
- added link l_if_slider_link, mass 0.00048911221771827; collision mesh filename=package://rohand_urdf_ros2/meshes_l/if_slider_link.STL; visual mesh filename=package://rohand_urdf_ros2/meshes_l/if_slider_link.STL
- added link l_lf_connecting_link, mass 0.000176980932045691; collision mesh filename=package://rohand_urdf_ros2/meshes_l/lf_connecting_link.STL; visual mesh filename=package://rohand_urdf_ros2/meshes_l/lf_connecting_link.STL
- added link l_lf_distal_link, mass 0.00262042947413116; collision mesh filename=package://rohand_urdf_ros2/meshes_l/lf_distal_link.STL; visual mesh filename=package://rohand_urdf_ros2/meshes_l/lf_distal_link.STL
- added link l_lf_proximal_link, mass 0.00136661208486985; collision mesh filename=package://rohand_urdf_ros2/meshes_l/lf_proximal_link.STL; visual mesh filename=package://rohand_urdf_ros2/meshes_l/lf_proximal_link.STL
- added link l_lf_slider_abpart_link, mass 0.000419595826532552; collision mesh filename=package://rohand_urdf_ros2/meshes_l/lf_slider_abpart_link.S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; visual mesh filename=package://rohand_urdf_ros2/meshes_l/lf_slider_abpart_link.S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
- added link l_lf_slider_link, mass 0.000510662528391611; collision mesh filename=package://rohand_urdf_ros2/meshes_l/lf_slider_link.STL; visual mesh filename=package://rohand_urdf_ros2/meshes_l/lf_slider_link.STL
- added link l_mf_connecting_link, mass 0.000216184518525667; collision mesh filename=package://rohand_urdf_ros2/meshes_l/mf_connecting_link.STL; visual mesh filename=package://rohand_urdf_ros2/meshes_l/mf_connecting_link.STL
- added link l_mf_distal_link, mass 0.0042269628029676; collision mesh filename=package://rohand_urdf_ros2/meshes_l/mf_distal_link.STL; visual mesh filename=package://rohand_urdf_ros2/meshes_l/mf_distal_link.STL
- added link l_mf_proximal_link, mass 0.00189508780970619; collision mesh filename=package://rohand_urdf_ros2/meshes_l/mf_proximal_link.STL; visual mesh filename=package://rohand_urdf_ros2/meshes_l/mf_proximal_link.STL
- added link l_mf_slider_abpart_link, mass 0.000419595848489683; collision mesh filename=package://rohand_urdf_ros2/meshes_l/mf_slider_abpart_link.S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; visual mesh filename=package://rohand_urdf_ros2/meshes_l/mf_slider_abpart_link.S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
- added link l_mf_slider_link, mass 0.000489112305392741; collision mesh filename=package://rohand_urdf_ros2/meshes_l/mf_slider_link.STL; visual mesh filename=package://rohand_urdf_ros2/meshes_l/mf_slider_link.STL
- added link l_rf_connecting_link, mass 0.000197692354337264; collision mesh filename=package://rohand_urdf_ros2/meshes_l/rf_connecting_link.STL; visual mesh filename=package://rohand_urdf_ros2/meshes_l/rf_connecting_link.STL
- added link l_rf_distal_link, mass 0.00422730983553646; collision mesh filename=package://rohand_urdf_ros2/meshes_l/rf_distal_link.STL; visual mesh filename=package://rohand_urdf_ros2/meshes_l/rf_distal_link.STL
- added link l_rf_proximal_link, mass 0.00154985371268108; collision mesh filename=package://rohand_urdf_ros2/meshes_l/rf_proximal_link.STL; visual mesh filename=package://rohand_urdf_ros2/meshes_l/rf_proximal_link.STL
- added link l_rf_slider_abpart_link, mass 0.000419595841745906; collision mesh filename=package://rohand_urdf_ros2/meshes_l/rf_slider_abpart_link.S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; visual mesh filename=package://rohand_urdf_ros2/meshes_l/rf_slider_abpart_link.S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
- added link l_rf_slider_link, mass 0.000489112303078988; collision mesh filename=package://rohand_urdf_ros2/meshes_l/rf_slider_link.STL; visual mesh filename=package://rohand_urdf_ros2/meshes_l/rf_slider_link.STL
- added link l_th_connecting_link, mass 0.000334843777726033; collision mesh filename=package://rohand_urdf_ros2/meshes_l/th_connecting_link.STL; visual mesh filename=package://rohand_urdf_ros2/meshes_l/th_connecting_link.STL
- added link l_th_distal_link, mass 0.00509494222453049; collision mesh filename=package://rohand_urdf_ros2/meshes_l/th_distal_link.STL; visual mesh filename=package://rohand_urdf_ros2/meshes_l/th_distal_link.STL
- added link l_th_proximal_link, mass 0.00501318922026079; collision mesh filename=package://rohand_urdf_ros2/meshes_l/th_proximal_link.STL; visual mesh filename=package://rohand_urdf_ros2/meshes_l/th_proximal_link.STL
- added link l_th_root_link, mass 0.00217782401907458; collision mesh filename=package://rohand_urdf_ros2/meshes_l/th_root_link.STL; visual mesh filename=package://rohand_urdf_ros2/meshes_l/th_root_link.STL
- added link l_th_slider_link, mass 0.000966918573679238; collision mesh filename=package://rohand_urdf_ros2/meshes_l/th_slider_link.STL; visual mesh filename=package://rohand_urdf_ros2/meshes_l/th_slider_link.STL
Joints:
- removed joint if_connecting_link
- removed joint if_distal_link
- removed joint if_proximal_link
- removed joint if_slider_abpart_link
- removed joint if_slider_link
- removed joint lf_connecting_link
- removed joint lf_distal_link
- removed joint lf_proximal_link
- removed joint lf_slider_abpart_link
- removed joint lf_slider_link
- removed joint mf_connecting_link
- removed joint mf_distal_link
- removed joint mf_proximal_link
- removed joint mf_slider_abpart_link
- removed joint mf_slider_link
- removed joint rf_connecting_link
- removed joint rf_distal_link
- removed joint rf_proximal_link
- removed joint rf_slider_abpart_link
- removed joint rf_slider_link
- removed joint th_connecting_link
- removed joint th_distal_link
- removed joint th_proximal_link
- removed joint th_root_link
- removed joint th_slider_link
- added joint l_if_connecting_link: type continuous, parent l_base_link, child l_if_connecting_link, origin xyz=-0.11976 0.03521 0.0067299 rpy=0 0 0, axis 0.082428 0.99278 -0.087177
- added joint l_if_distal_link: type continuous, parent l_if_proximal_link, child l_if_distal_link, origin xyz=-0.035776 0.0028401 -0.0014841 rpy=0 0 0, axis 0.082428 0.99278 -0.087177
- added joint l_if_proximal_link: type continuous, parent l_base_link, child l_if_proximal_link, origin xyz=-0.11211 0.037738 0.0020371 rpy=0 0 0, axis 0.082428 0.99278 -0.087177
- added joint l_if_slider_abpart_link: type continuous, parent l_if_slider_link, child l_if_slider_abpart_link, origin xyz=-0.02861 0.0058839 -0.00030477 rpy=0 0 0, axis 0.082734 0.99276 -0.087135
- added joint l_if_slider_link: type prismatic, parent l_base_link, child l_if_slider_link, origin xyz=-0.074396 0.026655 -0.0059032 rpy=0 0 0, axis 0.99655 -0.083049 0, limit lower=0 upper=0.019 effort=0 velocity=0
- added joint l_lf_connecting_link: type continuous, parent l_base_link, child l_lf_connecting_link, origin xyz=-0.11723 -0.027174 0.008365 rpy=0 0 0, axis -0.11759 0.98924 0.087085
- added joint l_lf_distal_link: type continuous, parent l_lf_proximal_link, child l_lf_distal_link, origin xyz=-0.031562 -0.0034532 -0.003392 rpy=0 0 0, axis -0.11759 0.98923 0.087106
- added joint l_lf_proximal_link: type continuous, parent l_base_link, child l_lf_proximal_link, origin xyz=-0.11032 -0.022406 0.0042916 rpy=0 0 0, axis -0.11759 0.98923 0.087106
- added joint l_lf_slider_abpart_link: type continuous, parent l_lf_slider_link, child l_lf_slider_abpart_link, origin xyz=-0.029209 4.0116E-05 0.00030326 rpy=0 0 0, axis -0.11759 0.98923 0.08715
- added joint l_lf_slider_link: type prismatic, parent l_base_link, child l_lf_slider_link, origin xyz=-0.070847 -0.024182 -0.0048997 rpy=0 0 0, axis 0.99301 0.11803 8.2704E-05, limit lower=0 upper=0.019 effort=0 velocity=0
- added joint l_mf_connecting_link: type continuous, parent l_base_link, child l_mf_connecting_link, origin xyz=-0.12334 0.014341 0.011366 rpy=0 0 0, axis 0.013244 0.99991 2.1054E-05
- added joint l_mf_distal_link: type continuous, parent l_mf_proximal_link, child l_mf_distal_link, origin xyz=-0.040851 0.00054126 -0.0035367 rpy=0 0 0, axis 0.013244 0.99991 2.1055E-05
- added joint l_mf_proximal_link: type continuous, parent l_base_link, child l_mf_proximal_link, origin xyz=-0.11587 0.017792 0.0069665 rpy=0 0 0, axis 0.013244 0.99991 4.2699E-05
- added joint l_mf_slider_abpart_link: type continuous, parent l_mf_slider_link, child l_mf_slider_abpart_link, origin xyz=-0.028951 0.0038841 0 rpy=0 0 0, axis 0.013228 0.99991 -7.2594E-05
- added joint l_mf_slider_link: type prismatic, parent l_base_link, child l_mf_slider_link, origin xyz=-0.076974 0.010077 -0.0016353 rpy=0 0 0, axis 0.99991 -0.013228 0.00010039, limit lower=0 upper=0.019 effort=0 velocity=0
- added joint l_rf_connecting_link: type continuous, parent l_base_link, child l_rf_connecting_link, origin xyz=-0.11723 -0.027174 0.008365 rpy=0 0 0, axis -0.05658 0.9984 2.102E-05
- added joint l_rf_distal_link: type continuous, parent l_rf_proximal_link, child l_rf_distal_link, origin xyz=-0.035766 -0.0020268 -0.0026198 rpy=0 0 0, axis -0.05658 0.9984 2.102E-05
- added joint l_rf_proximal_link: type continuous, parent l_base_link, child l_rf_proximal_link, origin xyz=-0.11364 -0.0022565 0.0062163 rpy=0 0 0, axis -0.05658 0.9984 2.102E-05
- added joint l_rf_slider_abpart_link: type continuous, parent l_rf_slider_link, child l_rf_slider_abpart_link, origin xyz=-0.029152 0.0018551 0 rpy=0 0 0, axis -0.056554 0.9984 -7.942E-05
- added joint l_rf_slider_link: type prismatic, parent l_base_link, child l_rf_slider_link, origin xyz=-0.074498 -0.0072492 -0.0023801 rpy=0 0 0, axis 0.9984 0.056554 9.5082E-05, limit lower=0 upper=0.019 effort=0 velocity=0
- added joint l_th_connecting_link: type continuous, parent l_th_slider_link, child l_th_connecting_link, origin xyz=-0.027697 0.024088 -0.010084 rpy=0 0 0, axis 0.21699 0.032029 -0.97565
- added joint l_th_distal_link: type continuous, parent l_th_proximal_link, child l_th_distal_link, origin xyz=-0.00010351 0.023735 -0.046849 rpy=0 -1.352 -0.032034, axis 0.21698 0.032029 -0.97565
- added joint l_th_proximal_link: type continuous, parent l_th_root_link, child l_th_proximal_link, origin xyz=-0.025097 0.021667 -0.015581 rpy=0.14303 1.3497 0.14655, axis 1 0 0
- added joint l_th_root_link: type revolute, parent l_base_link, child l_th_root_link, origin xyz=-0.024656 0.019554 -0.018266 rpy=0 0 0, axis -0.97616 0.01293 -0.21667, limit lower=0 upper=1.57 effort=0 velocity=0
- added joint l_th_slider_link: type prismatic, parent l_th_proximal_link, child l_th_slider_link, origin xyz=-0.0077 0.0027693 -0.00023667 rpy=0 -1.352 -0.032034, axis -0.76198 0.63028 -0.14877, limit lower=0 upper=0.01 effort=0 velocity=0
