Commit message: joints distinguish between left and right hands

File: urdf/rohand_right.urdf (robot description, URDF)
Before this commit: robot rohand_right, 26 links, 25 joints
Links:
- removed link base_link
- removed link if_connecting_link
- removed link if_distal_link
- removed link if_proximal_link
- removed link if_slider_abpart_link
- removed link if_slider_link
- removed link lf_connecting_link
- removed link lf_distal_link
- removed link lf_proximal_link
- removed link lf_slider_abpart_link
- removed link lf_slider_link
- removed link mf_connecting_link
- removed link mf_distal_link
- removed link mf_proximal_link
- removed link mf_slider_abpart_link
- removed link mf_slider_link
- removed link rf_connecting_link
- removed link rf_distal_link
- removed link rf_proximal_link
- removed link rf_slider_abpart_link
- removed link rf_slider_link
- removed link th_connecting_link
- removed link th_distal_link
- removed link th_proximal_link
- removed link th_root_link
- removed link th_slider_link
- added link r_base_link, mass 0.0941614898718946; collision mesh filename=package://rohand_urdf_ros2/meshes_r/base_link.STL; visual mesh filename=package://rohand_urdf_ros2/meshes_r/base_link.STL
- added link r_if_connecting_link, mass 0.000197689248381643; collision mesh filename=package://rohand_urdf_ros2/meshes_r/if_connecting_link.STL; visual mesh filename=package://rohand_urdf_ros2/meshes_r/if_connecting_link.STL
- added link r_if_distal_link, mass 0.00486631616894411; collision mesh filename=package://rohand_urdf_ros2/meshes_r/if_distal_link.STL; visual mesh filename=package://rohand_urdf_ros2/meshes_r/if_distal_link.STL
- added link r_if_proximal_link, mass 0.00154952958352476; collision mesh filename=package://rohand_urdf_ros2/meshes_r/if_proximal_link.STL; visual mesh filename=package://rohand_urdf_ros2/meshes_r/if_proximal_link.STL
- added link r_if_slider_abpart_link, mass 0.000526636346253179; collision mesh filename=package://rohand_urdf_ros2/meshes_r/if_slider_abpart_link.S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; visual mesh filename=package://rohand_urdf_ros2/meshes_r/if_slider_abpart_link.S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
- added link r_if_slider_link, mass 0.000489138281878773; collision mesh filename=package://rohand_urdf_ros2/meshes_r/if_slider_link.STL; visual mesh filename=package://rohand_urdf_ros2/meshes_r/if_slider_link.STL
- added link r_lf_connecting_link, mass 0.000176981602686642; collision mesh filename=package://rohand_urdf_ros2/meshes_r/lf_connecting_link.STL; visual mesh filename=package://rohand_urdf_ros2/meshes_r/lf_connecting_link.STL
- added link r_lf_distal_link, mass 0.00326999621591245; collision mesh filename=package://rohand_urdf_ros2/meshes_r/lf_distal_link.STL; visual mesh filename=package://rohand_urdf_ros2/meshes_r/lf_distal_link.STL
- added link r_lf_proximal_link, mass 0.00136677973237; collision mesh filename=package://rohand_urdf_ros2/meshes_r/lf_proximal_link.STL; visual mesh filename=package://rohand_urdf_ros2/meshes_r/lf_proximal_link.STL
- added link r_lf_slider_abpart_link, mass 0.000526636335571007; collision mesh filename=package://rohand_urdf_ros2/meshes_r/lf_slider_abpart_link.S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; visual mesh filename=package://rohand_urdf_ros2/meshes_r/lf_slider_abpart_link.S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
- added link r_lf_slider_link, mass 0.000489138222296884; collision mesh filename=package://rohand_urdf_ros2/meshes_r/lf_slider_link.STL; visual mesh filename=package://rohand_urdf_ros2/meshes_r/lf_slider_link.STL
- added link r_mf_connecting_link, mass 0.000216186298115104; collision mesh filename=package://rohand_urdf_ros2/meshes_r/mf_connecting_link.STL; visual mesh filename=package://rohand_urdf_ros2/meshes_r/mf_connecting_link.STL
- added link r_mf_distal_link, mass 0.00486610881870854; collision mesh filename=package://rohand_urdf_ros2/meshes_r/mf_distal_link.STL; visual mesh filename=package://rohand_urdf_ros2/meshes_r/mf_distal_link.STL
- added link r_mf_proximal_link, mass 0.00189501857338832; collision mesh filename=package://rohand_urdf_ros2/meshes_r/mf_proximal_link.STL; visual mesh filename=package://rohand_urdf_ros2/meshes_r/mf_proximal_link.STL
- added link r_mf_slider_abpart_link, mass 0.000526636368526203; collision mesh filename=package://rohand_urdf_ros2/meshes_r/mf_slider_abpart_link.S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; visual mesh filename=package://rohand_urdf_ros2/meshes_r/mf_slider_abpart_link.S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
- added link r_mf_slider_link, mass 0.000489138286069735; collision mesh filename=package://rohand_urdf_ros2/meshes_r/mf_slider_link.STL; visual mesh filename=package://rohand_urdf_ros2/meshes_r/mf_slider_link.STL
- added link r_rf_connecting_link, mass 0.000197689252304948; collision mesh filename=package://rohand_urdf_ros2/meshes_r/rf_connecting_link.STL; visual mesh filename=package://rohand_urdf_ros2/meshes_r/rf_connecting_link.STL
- added link r_rf_distal_link, mass 0.00486607601001256; collision mesh filename=package://rohand_urdf_ros2/meshes_r/rf_distal_link.STL; visual mesh filename=package://rohand_urdf_ros2/meshes_r/rf_distal_link.STL
- added link r_rf_proximal_link, mass 0.0015495346822944; collision mesh filename=package://rohand_urdf_ros2/meshes_r/rf_proximal_link.STL; visual mesh filename=package://rohand_urdf_ros2/meshes_r/rf_proximal_link.STL
- added link r_rf_slider_abpart_link, mass 0.000526636350514617; collision mesh filename=package://rohand_urdf_ros2/meshes_r/rf_slider_abpart_link.S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; visual mesh filename=package://rohand_urdf_ros2/meshes_r/rf_slider_abpart_link.S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
- added link r_rf_slider_link, mass 0.000489138255422532; collision mesh filename=package://rohand_urdf_ros2/meshes_r/rf_slider_link.STL; visual mesh filename=package://rohand_urdf_ros2/meshes_r/rf_slider_link.STL
- added link r_th_connecting_link, mass 0.000607798102631607; collision mesh filename=package://rohand_urdf_ros2/meshes_r/th_connecting_link.STL; visual mesh filename=package://rohand_urdf_ros2/meshes_r/th_connecting_link.STL
- added link r_th_distal_link, mass 0.00601772502419511; collision mesh filename=package://rohand_urdf_ros2/meshes_r/th_distal_link.STL; visual mesh filename=package://rohand_urdf_ros2/meshes_r/th_distal_link.STL
- added link r_th_proximal_link, mass 0.00501307756145889; collision mesh filename=package://rohand_urdf_ros2/meshes_r/th_proximal_link.STL; visual mesh filename=package://rohand_urdf_ros2/meshes_r/th_proximal_link.STL
- added link r_th_root_link, mass 0.00217782328356739; collision mesh filename=package://rohand_urdf_ros2/meshes_r/th_root_link.STL; visual mesh filename=package://rohand_urdf_ros2/meshes_r/th_root_link.STL
- added link r_th_slider_link, mass 0.000966927715708797; collision mesh filename=package://rohand_urdf_ros2/meshes_r/th_slider_link.STL; visual mesh filename=package://rohand_urdf_ros2/meshes_r/th_slider_link.STL
Joints:
- removed joint if_connecting_link
- removed joint if_distal_link
- removed joint if_proximal_link
- removed joint if_slider_abpart_link
- removed joint if_slider_link
- removed joint lf_connecting_link
- removed joint lf_distal_link
- removed joint lf_proximal_link
- removed joint lf_slider_abpart_link
- removed joint lf_slider_link
- removed joint mf_connecting_link
- removed joint mf_distal_link
- removed joint mf_proximal_link
- removed joint mf_slider_abpart_link
- removed joint mf_slider_link
- removed joint rf_connecting_link
- removed joint rf_distal_link
- removed joint rf_proximal_link
- removed joint rf_slider_abpart_link
- removed joint rf_slider_link
- removed joint th_connecting_link
- removed joint th_distal_link
- removed joint th_proximal_link
- removed joint th_root_link
- removed joint th_slider_link
- added joint r_if_connecting_link: type continuous, parent r_base_link, child r_if_connecting_link, origin xyz=-0.12029 -0.028806 0.0072922 rpy=0 0 0, axis -0.082428 0.99278 0.087177
- added joint r_if_distal_link: type continuous, parent r_if_proximal_link, child r_if_distal_link, origin xyz=-0.035776 -0.0028401 -0.0014841 rpy=0 0 0, axis -0.082428 0.99278 0.087177
- added joint r_if_proximal_link: type continuous, parent r_base_link, child r_if_proximal_link, origin xyz=-0.11324 -0.024137 0.0032314 rpy=0 0 0, axis -0.082428 0.99278 0.087177
- added joint r_if_slider_abpart_link: type continuous, parent r_if_slider_link, child r_if_slider_abpart_link, origin xyz=-0.029189 0.0010654 0.00030518 rpy=0 0 0, axis -0.082734 0.99276 0.087135
- added joint r_if_slider_link: type prismatic, parent r_base_link, child r_if_slider_link, origin xyz=-0.074396 -0.026655 -0.0059032 rpy=0 0 0, axis 0.99655 0.083049 0, limit lower=0 upper=0.019 effort=0 velocity=0
- added joint r_lf_connecting_link: type continuous, parent r_base_link, child r_lf_connecting_link, origin xyz=-0.11647 0.033555 0.0078033 rpy=0 0 0, axis 0.11759 0.98924 -0.087085
- added joint r_lf_distal_link: type continuous, parent r_lf_proximal_link, child r_lf_distal_link, origin xyz=-0.031562 0.0034532 -0.003392 rpy=0 0 0, axis 0.11759 0.98923 -0.087106
- added joint r_lf_proximal_link: type continuous, parent r_base_link, child r_lf_proximal_link, origin xyz=-0.10871130258864 0.0359583660197833 0.00309824490260681 rpy=0 0 0, axis 0.117591058209323 0.989234457465869 -0.0871064359930968
- added joint r_lf_slider_abpart_link: type continuous, parent r_lf_slider_link, child r_lf_slider_abpart_link, origin xyz=-0.0283858043783233 0.00688449840682251 -0.000306788289491815 rpy=0 0 0, axis 0.117590610595967 0.989230669602698 -0.0871500465694956
- added joint r_lf_slider_link: type prismatic, parent r_base_link, child r_lf_slider_link, origin xyz=-0.0708466334619896 0.0241824111749996 -0.00489967270216645 rpy=0 0 0, axis 0.993009723934899 -0.118032543523823 8.27044911595336E-05, limit lower=0 upper=0.019 effort=0 velocity=0
- added joint r_mf_connecting_link: type continuous, parent r_base_link, child r_mf_connecting_link, origin xyz=-0.12342 -0.0078912 0.011366 rpy=0 0 0, axis -0.013244 0.99991 -2.1054E-05
- added joint r_mf_distal_link: type continuous, parent r_mf_proximal_link, child r_mf_distal_link, origin xyz=-0.040851 -0.00054126 -0.0035364 rpy=0 0 0, axis -0.013244 0.99991 -2.1055E-05
- added joint r_mf_proximal_link: type continuous, parent r_base_link, child r_mf_proximal_link, origin xyz=-0.11605 -0.0040932 0.0069659 rpy=0 0 0, axis -0.013244 0.99991 -4.2699E-05
- added joint r_mf_slider_abpart_link: type continuous, parent r_mf_slider_link, child r_mf_slider_abpart_link, origin xyz=-0.029044 0.0031153 0 rpy=0 0 0, axis -0.013228 0.99991 7.2594E-05
- added joint r_mf_slider_link: type prismatic, parent r_base_link, child r_mf_slider_link, origin xyz=-0.076974 -0.010077 -0.0016353 rpy=0 0 0, axis 0.99991 0.013228 0.00010039, limit lower=0 upper=0.019 effort=0 velocity=0
- added joint r_rf_connecting_link: type continuous, parent r_base_link, child r_rf_connecting_link, origin xyz=-0.1204851022382 0.0126604995038233 0.0106153804877178 rpy=0 0 0, axis 0.0565797489260885 0.99839808271532 -2.10198201110756E-05
- added joint r_rf_distal_link: type continuous, parent r_rf_proximal_link, child r_rf_distal_link, origin xyz=-0.035766 0.0020268 -0.0026198 rpy=0 0 0, axis 0.05658 0.9984 -2.102E-05
- added joint r_rf_proximal_link: type continuous, parent r_base_link, child r_rf_proximal_link, origin xyz=-0.11287 0.015935 0.0062161 rpy=0 0 0, axis 0.05658 0.9984 -2.102E-05
- added joint r_rf_slider_abpart_link: type continuous, parent r_rf_slider_link, child r_rf_slider_abpart_link, origin xyz=-0.028756 0.0051336 0 rpy=0 0 0, axis 0.056554 0.9984 7.942E-05
- added joint r_rf_slider_link: type prismatic, parent r_base_link, child r_rf_slider_link, origin xyz=-0.074498 0.0072492 -0.0023801 rpy=0 0 0, axis 0.9984 -0.056554 9.5082E-05, limit lower=0 upper=0.019 effort=0 velocity=0
- added joint r_th_connecting_link: type continuous, parent r_th_slider_link, child r_th_connecting_link, origin xyz=-0.026144 -0.020984 -0.0010258 rpy=0 0 0, axis -0.21699 0.032029 0.97565
- added joint r_th_distal_link: type continuous, parent r_th_proximal_link, child r_th_distal_link, origin xyz=-0.049076 -0.023254 0.004868 rpy=0 0 0, axis -0.21698 0.032029 0.97565
- added joint r_th_proximal_link: type continuous, parent r_th_root_link, child r_th_proximal_link, origin xyz=-0.025097 -0.021667 -0.015581 rpy=0 0 0, axis -0.21699 -0.032029 0.97565
- added joint r_th_root_link: type revolute, parent r_base_link, child r_th_root_link, origin xyz=-0.024656 -0.019554 -0.018266 rpy=0 0 0, axis 0.97616 0.01293 0.21667, limit lower=0 upper=1.57 effort=0 velocity=0
- added joint r_th_slider_link: type prismatic, parent r_th_proximal_link, child r_th_slider_link, origin xyz=-0.0053401 -0.0053494 0.0068801 rpy=0 0 0, axis -0.76198 -0.63028 -0.14877, limit lower=0 upper=0.01 effort=0 velocity=0
